File: hardware/Console_Lights.kicad_pcb (KiCad board)
At the start: 2 copper layers, 65.6 x 77.6 mm, 46 parts, among them J504 JST_Conn, J505 JST_Conn, J506 JST_Conn, J507 JST_Conn, J508 JST_Conn, J509 JST_Conn, J510 JST_Conn, J511 JST_Conn, J512 JST_Conn, J513 JST_Conn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

Commit message: shcematic/routing updates, add fab notes
Parts:
- added REF**: GND_Stitch_Via, ConsoleLights:GND_Stitch_Via, F.Cu at (139.1, 68.8)
- added REF**: GND_Stitch_Via, ConsoleLights:GND_Stitch_Via, F.Cu at (125.2, 90.2)
- added REF**: FAB_NOTES, ConsoleLights:FAB_NOTES, F.Cu at (12.0, 12.0)
- added REF**: STACKUP, ConsoleLights:STACKUP, F.Cu at (267.4, 12.0)
- added REF**: GND_Stitch_Via, ConsoleLights:GND_Stitch_Via, F.Cu at (152.9, 90.2)
- added REF**: GND_Stitch_Via, ConsoleLights:GND_Stitch_Via, F.Cu at (135.0, 99.8)
- moved U106 0.47 mm to (139.1, 96.5)
Routing:
- net /LATCH: track 5.34 -> 39.0 mm, vias 0 -> 1
- net Net-(U102-Pad14): track 34.3 -> 36.1 mm
- net /SWITCH_2: track 62.3 -> 63.5 mm
- net +5V: track 61.8 -> 62.5 mm
- net /SWITCH_9: track 62.2 -> 62.8 mm

Commit message: layout updates
Parts:
- added G***: LOGO, ConsoleLights:TARDIS, F.Cu at (154.8, 124.5)
- added REF**: GND_Stitch_Via, ConsoleLights:GND_Stitch_Via, F.Cu at (139.1, 117.0)
- SW501: footprint ConsoleLights:Panasonic_Tac_Switch_EVQ-Q2K03W -> ConsoleLights:CK_PTS645_Tac_Switch
- moved SW501 0.25 mm to (139.1, 139.2), turned to 180 degrees
Routing:
- net /MODE: track 16.5 -> 17.4 mm
- net /SWITCH_3: track 40.4 -> 41.1 mm
- net /SWITCH_2: track 63.5 -> 64.1 mm
- net /SWITCH_9: track 62.8 -> 63.4 mm
- net /LED_8: track 28.2 -> 27.6 mm
Other:
- board text added: "Lights of Rassilon"
- board text added: "NOCTIVORE"

Commit message: add seal, prints, production files
Parts:
- added G***: LOGO, ConsoleLights:SEAL_OF_RASSILON, F.Cu at (123.5, 124.5)
Other:
- board text added: "0"
- board text added: "1"
- board text added: "2"
- board text added: "3"
- board text added: "4"
- board text added: "5"
- board text added: "6"
- board text added: "7"
- board text added: "8"
- board text added: "9"
